Commit message: adding stl_files to image_labeling

File: image_labeling/urdf/atlas2.urdf (robot description, URDF)
Before this commit: robot ATLCASCAR2, 1 links, 0 joints
Links:
- link map: geometry visual mesh filename=package://image_labeling/stl_files/atlas2.STL

Commit message: debug + dependencies folder

File: image_labeling/urdf/atlas2.urdf (robot description, URDF)
Before this commit: robot ATLCASCAR2, 1 links, 0 joints
Links:
- link map: geometry visual mesh filename=package://free_space_detection/stl_files/atlas2.STL
